File: BatteryInterconnects.kicad_pcb (KiCad board)
At the start: 2 copper layers, 347.5 x 31 mm, 4 parts, among them J1 Conn_01x02_Socket, J2 Conn_01x02_Socket, J3 Conn_01x02_Pin, J4 Conn_01x02_Pin

Commit message: Tweaks and Production files
Parts:
- J1, J2: footprint Connector_AMASS:AMASS_XT30PW-F_1x02_P2.50mm_Horizontal -> Connector_AMASS:AMASS_XT30U-F_1x02_P5.0mm_Vertical
- J3, J4: footprint Connector_AMASS:AMASS_XT30PW-M_1x02_P2.50mm_Horizontal -> Connector_AMASS:AMASS_XT30U-M_1x02_P5.0mm_Vertical
- moved J3 15.0 mm to (346.3, 133.0), turned to 90 degrees
- moved J1 10.3 mm to (23.6, 133.0)
- moved J2 10.3 mm to (23.6, 149.0)
- moved J4 8.24 mm to (365.5, 128.2)
Other:
- board size 347.5 x 31 mm -> 350.5 x 31 mm
